File: powerwatch/electron_rev_3/hardware/plugwatch.brd (EAGLE design)
At the start: 57.1 x 93 mm, 125 parts, among them J1 DM3AT-SF-PEJM5, J2 TC2030-JLINK-NL, U1 BGA725L6-ALT, U10 SIP32510, U11 SIP32510, U12 SIP32510, U13 SIP32510, U14 MPU-9250, U15 OPA322AIDBVT, U2 SAFFB1G56KB0F0A, U3 ISL29035, U4 MAX-M8, U5 MAX740XESA, U6 SIP32510, U7 NRF51822QF, U8 OPA322AIDBVT, U9 SIP32510, X1 32.768k, X2 16MHz

Commit message: pushing for production
Parts:
- removed L6: 27uH, SparkFun-Passives:1X02
- added IND, IND1: TEST_POINT_0.040IN, headers:TESTPOINT_0.040IN
Connections:
- net GND: now also IND1.TESTPOINT
- net INDUCTIVE_ANTENNA: now also IND.TESTPOINT; no longer L6.2
Other:
- board text added: "(ON, ON)"
- board text removed: "(on, on)"
Changed lines of the file:
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@@
 <?xml version="1.0" encoding="utf-8"?>
 <!DOCTYPE eagle SYSTEM "eagle.dtd">
-<eagle version="8.5.0">
+<eagle version="8.7.1">
 <drawing>
 <settings>
-<setting alwaysvectorfont="yes"/>
+<setting alwaysvectorfont="no"/>
 <setting verticaltext="up"/>
 </settings>
@@
 <text x="52.832" y="20.574" size="1.27" layer="25" font="vector" ratio="12" align="bottom-center">AUDIO</text>
 <text x="52.832" y="37.338" size="0.8128" layer="25" font="vector" ratio="12" rot="R90" align="bottom-center">AUDIO_PWR_EN</text>
-<text x="53.848" y="68.326" size="0.8128" layer="25" font="vector" ratio="12" rot="R90" align="bottom-center">IND_ANT</text>
+<text x="53.594" y="68.326" size="0.8128" layer="25" font="vector" ratio="12" rot="R90" align="bottom-center">IND_ANT</text>
 <text x="54.61" y="55.118" size="1.016" layer="25" font="vector" ratio="12" align="bottom-center">VCC</text>
 <wire x1="57.15" y1="0" x2="57.15" y2="42.037" width="0.0254" layer="20"/>
@@
 <text x="9.144" y="20.32" size="1.27" layer="25" font="vector" ratio="12" align="bottom-center">SD CARD</text>
 <text x="47.752" y="73.914" size="1.778" layer="25" font="vector" ratio="12">APN</text>
-<text x="47.752" y="72.644" size="0.8128" layer="25" font="vector" ratio="12">(on, on)</text>
+<text x="47.752" y="72.644" size="0.8128" layer="25" font="vector" ratio="12">(ON, ON)</text>
 </plain>
 <attributes>
@@
 <attribute name="NAME" x="33.02" y="39.624" size="1.016" layer="26" font="vector" ratio="12" rot="MR0" align="bottom-center"/>
 </element>
-<element name="L6" library="SparkFun-Passives" package="1X02" value="27uH" x="55.372" y="60.198" smashed="yes" rot="R90">
-<attribute name="DIGIKEY" value="445-173093-ND" x="55.372" y="60.198" size="1.778" layer="27" rot="R90" display="off"/>
-<attribute name="NAME" x="55.8292" y="64.4398" size="1.016" layer="25" font="vector" ratio="12" rot="R90"/>
-<attribute name="VALUE" x="58.547" y="58.928" size="1.27" layer="27" rot="R90"/>
-</element>
 <element name="MK1" library="microphones" package="MIC_AOM-4546P-R" value="AOM-4546P-R" x="52.07" y="22.225" locked="yes" smashed="yes" rot="MR0">
 <attribute name="DIGIKEY" value="668-1224-ND" x="52.07" y="22.225" size="1.778" layer="27" display="off"/>
@@
 <attribute name="NAME" x="55.626" y="76.581" size="1.016" layer="25" font="vector" ratio="12" rot="R180" align="bottom-center"/>
 <attribute name="VALUE" x="56.769" y="74.676" size="1.016" layer="27" font="vector" ratio="12" rot="R90" align="bottom-center"/>
+</element>
+<element name="IND" library="headers" package="TESTPOINT_0.040IN" value="TEST_POINT_0.040IN" x="55.372" y="62.23" smashed="yes">
+<attribute name="DIGIKEY" value="5001K-ND" x="55.372" y="62.23" size="1.778" layer="27" display="off"/>
+<attribute name="NAME" x="55.88" y="59.436" size="1.016" layer="25" font="vector" ratio="12" rot="R90" align="bottom-center"/>
+<attribute name="VALUE" x="55.372" y="59.69" size="1.016" layer="27" font="vector" ratio="12" align="bottom-center"/>
+</element>
+<element name="IND1" library="headers" package="TESTPOINT_0.040IN" value="TEST_POINT_0.040IN" x="55.372" y="70.358" smashed="yes">
+<attribute name="DIGIKEY" value="5001K-ND" x="55.372" y="70.358" size="1.778" layer="27" display="off"/>
+<attribute name="NAME" x="55.88" y="67.31" size="1.016" layer="25" font="vector" ratio="12" rot="R90" align="bottom-center"/>
+<attribute name="VALUE" x="55.372" y="67.818" size="1.016" layer="27" font="vector" ratio="12" align="bottom-center"/>
 </element>
 </elements>
@@
 <wire x1="29.464" y1="2.54" x2="56.134" y2="2.54" width="0.3048" layer="1"/>
 <wire x1="3.81" y1="92.202" x2="0.762" y2="89.154" width="0.3048" layer="1"/>
-<wire x1="51.435" y1="64.262" x2="51.435" y2="68.199" width="0.3048" layer="1"/>
-<wire x1="51.435" y1="68.199" x2="56.388" y2="73.152" width="0.3048" layer="1"/>
+<wire x1="51.435" y1="64.262" x2="51.435" y2="68.961" width="0.3048" layer="1"/>
+<wire x1="51.435" y1="68.961" x2="56.388" y2="73.66" width="0.3048" layer="1"/>
 <wire x1="54.102" y1="92.202" x2="27.178" y2="92.202" width="0.3048" layer="1"/>
-<wire x1="56.388" y1="73.152" x2="56.388" y2="89.916" width="0.3048" layer="1"/>
+<wire x1="56.388" y1="73.66" x2="56.388" y2="89.916" width="0.3048" layer="1"/>
 <wire x1="56.388" y1="89.916" x2="54.102" y2="92.202" width="0.3048" layer="1"/>
 <wire x1="6.35" y1="51.562" x2="7.366" y2="51.562" width="0.3048" layer="1"/>
@@
 <wire x1="12.81025" y1="42.738" x2="13.65" y2="42.738" width="0.254" layer="1"/>
 <wire x1="13.208" y1="39.624" x2="13.97" y2="40.386" width="0.508" layer="16"/>
-<wire x1="13.363" y1="24.638" x2="10.668" y2="24.638" width="0.8128" layer="1"/>
+<wire x1="13.617" y1="24.638" x2="10.668" y2="24.638" width="0.8128" layer="1"/>
 <wire x1="13.65" y1="42.738" x2="13.777" y2="42.611" width="0.254" layer="1"/>
 <wire x1="13.777" y1="42.611" x2="13.97" y2="42.418" width="0.3048" layer="1"/>
@@
 <wire x1="14.8504" y1="8.1316" x2="14.8504" y2="8.797" width="0.2032" layer="16"/>
 <wire x1="14.8504" y1="8.797" x2="14.1732" y2="9.6012" width="0.2032" layer="16"/>
-<wire x1="15.101" y1="22.9" x2="13.363" y2="24.638" width="0.8128" layer="1"/>
+<wire x1="15.101" y1="22.9" x2="13.617" y2="24.638" width="0.8128" layer="1"/>
 <wire x1="15.235" y1="7.747" x2="14.8504" y2="8.1316" width="0.2032" layer="16"/>
 <wire x1="15.748" y1="7.747" x2="15.235" y2="7.747" width="0.2032" layer="16"/>
@@
 <via x="50.292" y="71.628" extent="1-16" drill="0.3048"/>
 <via x="52.832" y="71.628" extent="1-16" drill="0.3048"/>
+<contactref element="IND1" pad="TESTPOINT"/>
 </signal>
 <signal name="GPS_PWR_EN">
@@
 <signal name="INDUCTIVE_ANTENNA">
 <contactref element="JP1" pad="1"/>
-<contactref element="L6" pad="2"/>
-<wire x1="53.213" y1="64.262" x2="54.737" y2="62.738" width="0.3048" layer="1"/>
-<wire x1="54.737" y1="62.738" x2="55.372" y2="62.738" width="0.3048" layer="1"/>
+<contactref element="IND" pad="TESTPOINT"/>
+<wire x1="55.372" y1="62.23" x2="53.34" y2="64.262" width="0.1524" layer="1"/>
+<wire x1="53.34" y1="64.262" x2="53.213" y2="64.262" width="0.1524" layer="1"/>
 </signal>
 <signal name="LED">
