File: powerwatch/electron_rev_3/hardware/plugwatch.sch (EAGLE design)
At the start: 110 parts, among them J1 DM3AT-SF-PEJM5, J2 TC2030-JLINK-NL, U1 BGA725L6-ALT, U10 SIP32510, U11 SIP32510, U12 SIP32510, U13 SIP32510, U2 SAFFB1G56KB0F0A, U3 ISL29035, U4 MAX-M8, U5 MAX740XESA, U6 MPU-9250, U7 NRF51822QF, U8 OPA322AIDBVT, U9 SIP32510, X1 ABS05-32.768KHZ-9-T, X2 16MHz

Commit message: Tried to address a lot of #2
Still need prefilter audio output

Need a check over 60hz antenna stuff
Parts:
- added JP1: JUMPER-3SMD, SparkFun-Passives:JUMPER-3SMD
- added L6: (no value), SparkFun-Passives:JUMPER-2PTH
- added R26: 100k, passives:RESISTOR0402_RES
- added R27: 10k, passives:RESISTOR0402_RES
- added R28: 487k, passives:RESISTOR0402_RES
- added TP18, TP26: TEST_POINT_0.040IN, headers:TEST_POINT_0.040IN
- added U14: MPU-9250, chips:MPU-9250
- added U15: OPA322AIDBVT, opamps:OPA322AIDBVT
- C27: device passives:CAPACITOR0402_CAP -> passives:CAPACITOR0805_CAP
- U6: value MPU-9250 -> SIP32510; device Testing:MPU-9250 -> chips:SIP32510; DIGIKEY 1428-1019-1-ND -> (none)
Connections:
- removed net REGOUT: C18.1, U6.REGOUT
- removed net SD_ENABLE_POWER: R17.1, U12.EN
- new net 60HZ_AMP: ASSY1.B3, R28.2, U15.OUT
- new net 60HZ_TRACE: JP1.3
- new net INDUCTIVE_ANTENNA: JP1.1, L6.2
- new net N$19: C18.1, U14.REGOUT
- new net N$23: R27.2, R28.1, U15.-IN
- new net N$30: JP1.2, U15.+IN
- new net SD_ENABLE: ASSY1.D5, R17.1, U12.EN
- new net SENSORS_PWR_EN: R26.1, U6.EN
- new net VCC_SENSORS: C13.1, C17.1, C19.1, R10.2, R11.2, R8.2, R9.2, U14.!CS, U14.VDD, U14.VDDIO, U3.VDD, U6.VLOAD
- net !IMU_INT: now also U14.INT; no longer U6.INT
- net GND: now also R27.1, TP26.TESTPOINT, U14.AD0/MISO, U14.FSYNC, U14.GND, U15.V-; no longer U6.AD0/SDO, U6.FSYNC
- net SENSORS_SCL: now also U14.SCLK; no longer U6.SCL/SCLK
- net SENSORS_SDA: now also U14.SDA/MOSI; no longer U6.SDA/SDI
- net VCC: now also R26.2, TP18.TESTPOINT, U15.V+, U6.VSUPP; no longer C13.1, C17.1, C19.1, R10.2, R11.2, R8.2, R9.2, U3.VDD, U6.!CS, U6.VDD, U6.VDDIO
Other:
- moved on the sheet: C13, C17, C18, C19, R10, R11, R8, R9, TP19, TP20, TP21, TP22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

Commit message: add plugwatch last fixes
Parts:
- added TP27, TP28: TEST_POINT_0.040IN, headers:TEST_POINT_0.040IN
Connections:
- new net B0: ASSY1.B0, TP28.TESTPOINT
- net A_MIC_OUT: now also TP27.TESTPOINT

Commit message: add production files
Parts:
- A2: DESCRIPTION (none) -> PATCH ANT GPS/GLO CP SMD; MANUFACTURER (none) -> Yageo; MPN (none) -> ANT1818B00BT1516S
- ASSY1: DESCRIPTION (none) -> 18 Position header; MANUFACTURER (none) -> Sullins; MPN (none) -> PPPC181LFBN-RC
- C1: DESCRIPTION (none) -> CAP CER 0.8PF 50V C0G/NP0 0402; MANUFACTURER (none) -> Murata; MPN (none) -> GRM1555C1HR80BA01D
- C10: DESCRIPTION (none) -> CAP CER 2200PF 25V 10% X7R 0402; MANUFACTURER (none) -> Murata; MPN (none) -> GRM155R71E222KA01D
- C11, C12, C13: DESCRIPTION (none) -> CAP CER 10000PF 50V X7R 0402; MANUFACTURER (none) -> Murata; MPN (none) -> GRM155R71H103JA88D
- C14: DESCRIPTION (none) -> CAP CER 0.047UF 16V X7R 0402; MANUFACTURER (none) -> Murata; MPN (none) -> GRM155R71C473KA01J
- C15, C16, C17, C18, C19, C20, C21: DESCRIPTION (none) -> CAP CER 0.1UF 10V X7R 0402; MANUFACTURER (none) -> Murata; MPN (none) -> GRM155R71A104JA01D
- C2: DESCRIPTION (none) -> CAP CER RF 4.4PF 50V +/-0.1 PF C; MANUFACTURER (none) -> KEMET; MPN (none) -> CBR06C449B5GAC
- C22: DESCRIPTION (none) -> CAP CER 1UF 10V X7S 0402; MANUFACTURER (none) -> Murata; MPN (none) -> GRM155C71A105KE11D
- C23, C24: DESCRIPTION (none) -> CAP TANT 2.2UF 16V 10% 1206; MANUFACTURER (none) -> Vishay; MPN (none) -> 293D225X9016A2TE3
- C25, C26: DESCRIPTION (none) -> CAP CER 4.7UF 6.3V X5R 0402; MANUFACTURER (none) -> TDK; MPN (none) -> C1005X5R0J475K050BC
- C27: DESCRIPTION (none) -> CAP CER 10UF 10V X7R 0805; MANUFACTURER (none) -> Murata; MPN (none) -> GRM21BR71A106ME51L
- C28: DESCRIPTION (none) -> CAP TANT 10UF 20V 10% 1206; MANUFACTURER (none) -> AVX; MPN (none) -> F951D106KSAAQ2
- C3, C4, C5, C6: DESCRIPTION (none) -> CAP CER 12PF 50V C0G/NP0 0402; MANUFACTURER (none) -> Murata; MPN (none) -> GRM1555C1H120GA01D
- C7: DESCRIPTION (none) -> CAP CER 330PF 50V C0G/NP0 0402; MANUFACTURER (none) -> Murata; MPN (none) -> GRM1555C1H331FA01D
- C8, C9: DESCRIPTION (none) -> CAP CER 1000PF 100V 10% X7R 0402; MANUFACTURER (none) -> Murata; MPN (none) -> GRM155R72A102KA01D
- D1, D2, D3: value LED0603 -> BLUE
- L1: DESCRIPTION (none) -> FIXED IND 5.6NH 1.77A 40 MOHM; MANUFACTURER (none) -> Murata; MPN (none) -> LQW15AN5N6B80D
- L2: DESCRIPTION (none) -> FIXED IND 15NH 320MA 460 MOHM; MANUFACTURER (none) -> Taiyo Yuden; MPN (none) -> HK100515NJ-T
- L3: DESCRIPTION (none) -> FIXED IND 10UH 50MA 900 MOHM SMD; MANUFACTURER (none) -> Murata; MPN (none) -> LQM18FN100M00D
- L4, L5: DESCRIPTION (none) -> FERRITE BEAD 1 KOHM 0402 1LN; MANUFACTURER (none) -> Murata; MPN (none) -> BLM15HD102SN1D
- L6: value (none) -> 27uH; DIGIKEY (none) -> 445-173093-ND
- R1: DESCRIPTION (none) -> RES SMD 49.9 OHM 1% 1/10W 0603; MANUFACTURER (none) -> Vishay; MPN (none) -> CRCW060349R9FKTA
- R10, R11, R12, R13, R14, R27, R8, R9: DESCRIPTION (none) -> RES SMD 10K OHM 1% 1/16W 0402; MANUFACTURER (none) -> Stackpole Electronics; MPN (none) -> RMCF0402FT10K0
- R15: DESCRIPTION (none) -> RES SMD 12K OHM 1% 1/16W 0402; MANUFACTURER (none) -> Stackpole Electronics; MPN (none) -> RMCF0402FT12K0
- R16, R17, R18, R19, R20, R21, R26: DESCRIPTION (none) -> RES SMD 100K OHM 1% 1/16W 0402; MANUFACTURER (none) -> Samsung; MPN (none) -> RC1005F104CS
- R2, R3: DESCRIPTION (none) -> RES SMD 150 OHM 1% 1/16W 0402; MANUFACTURER (none) -> Stackpole Electronics; MPN (none) -> RMCF0402FT150R
- R22, R23, R24: DESCRIPTION (none) -> RES SMD 100K OHM 1% 1/10W 0603; MANUFACTURER (none) -> Vishay; MPN (none) -> CRCW0603100KFKEB
- R25: DESCRIPTION (none) -> RES SMD 270K OHM 1% 1/10W 0603; MANUFACTURER (none) -> Vishay; MPN (none) -> CRCW0603270KFKEA
- R28: DESCRIPTION (none) -> RES 487K OHM 1/16W 1% 0402 SMD; MANUFACTURER (none) -> Yageo; MPN (none) -> RC0402FR-07487KL
- R4, R5, R6: DESCRIPTION (none) -> RES SMD 1K OHM 1% 1/16W 0402; MANUFACTURER (none) -> Stackpole Electronics; MPN (none) -> RMCF0402FT1K00
- R7: DESCRIPTION (none) -> RES SMD 3.48K OHM 1% 1/10W 0603; MANUFACTURER (none) -> Vishay; MPN (none) -> CRCW06033K48FKEA
- U1: DESCRIPTION (none) -> IC AMP MMIC RF LNA 20DB TSLP-6; MANUFACTURER (none) -> Infineon; MPN (none) -> BGA725L6E6327FTSA1
- U4: DESCRIPTION (none) -> IC RECEIVER GPS/GNSS 18LCC; MANUFACTURER (none) -> u-blox; MPN (none) -> MAX-M8Q-0
- X1: value ABS05-32.768KHZ-9-T -> 32.768k
- X2: DESCRIPTION (none) -> CRYSTAL 16.0000MHZ 8PF SMD; MANUFACTURER (none) -> TXC; MPN (none) -> 8Y-16.000MAAV-T
