File: powerwatch/electron_rev_3/hardware/plugwatch.sch (EAGLE design)
At the start: 124 parts, among them J1 DM3AT-SF-PEJM5, J2 TC2030-JLINK-NL, U1 BGA725L6-ALT, U10 SIP32510, U11 SIP32510, U12 SIP32510, U13 SIP32510, U14 MPU-9250, U15 OPA322AIDBVT, U2 SAFFB1G56KB0F0A, U3 ISL29035, U4 MAX-M8, U5 MAX740XESA, U6 SIP32510, U7 NRF51822QF, U8 OPA322AIDBVT, U9 SIP32510, X1 32.768k, X2 16MHz

Commit message: pushing for production
Parts:
- removed L6: 27uH, SparkFun-Passives:JUMPER-2PTH
- added IND, IND1: TEST_POINT_0.040IN, headers:TEST_POINT_0.040IN
Connections:
- net GND: now also IND1.TESTPOINT
- net INDUCTIVE_ANTENNA: now also IND.TESTPOINT; no longer L6.2
Changed lines of the file:
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@@
 <?xml version="1.0" encoding="utf-8"?>
 <!DOCTYPE eagle SYSTEM "eagle.dtd">
-<eagle version="8.5.0">
+<eagle version="8.7.1">
 <drawing>
 <settings>
-<setting alwaysvectorfont="yes"/>
+<setting alwaysvectorfont="no"/>
 <setting verticaltext="up"/>
 </settings>
-<grid distance="0.1" unitdist="inch" unit="inch" style="lines" multiple="1" display="yes" altdistance="0.05" altunitdist="inch" altunit="inch"/>
+<grid distance="0.1" unitdist="inch" unit="inch" style="lines" multiple="1" display="no" altdistance="0.01" altunitdist="inch" altunit="inch"/>
 <layers>
 <layer number="1" name="Top" color="4" fill="1" visible="no" active="no"/>
@@
 <attribute name="MPN" value="BLM15HD102SN1D"/>
 </part>
-<part name="L6" library="SparkFun-Passives" deviceset="JUMPER-2" device="PTH" value="27uH">
-<attribute name="DIGIKEY" value="445-173093-ND"/>
-</part>
 <part name="MK1" library="microphones" deviceset="AOM-4546P-R" device=""/>
 <part name="P+10" library="supply1" library_urn="urn:adsk.eagle:library:371" deviceset="VCC" device=""/>
@@
 </part>
 <part name="GND13" library="umich" deviceset="GND" device=""/>
+<part name="IND" library="headers" deviceset="TEST_POINT_0.040IN" device=""/>
+<part name="IND1" library="headers" deviceset="TEST_POINT_0.040IN" device=""/>
+<part name="GND42" library="supply1" library_urn="urn:adsk.eagle:library:371" deviceset="GND" device=""/>
 </parts>
 <sheets>
@@
 <attribute name="DIGIKEY" x="168.91" y="130.81" size="1.27" layer="96" display="off"/>
 </instance>
-<instance part="L6" gate="A" x="157.48" y="55.88" rot="MR180">
-<attribute name="DIGIKEY" x="157.48" y="55.88" size="1.016" layer="96" rot="MR180" align="bottom-center" display="off"/>
-</instance>
 <instance part="P+15" gate="VCC" x="119.38" y="78.74"/>
 <instance part="P+1" gate="VCC" x="175.26" y="177.8"/>
@@
 </instance>
 <instance part="U9" gate="G$1" x="99.06" y="71.12" rot="R180"/>
+<instance part="IND" gate="G$1" x="157.48" y="58.42"/>
+<instance part="IND1" gate="G$1" x="157.48" y="53.34"/>
+<instance part="GND42" gate="1" x="162.56" y="48.26" rot="MR0"/>
 </instances>
 <busses>
@@
 <pinref part="U15" gate="U1" pin="V-"/>
 <wire x1="203.2" y1="58.42" x2="203.2" y2="55.88" width="0.1524" layer="91"/>
+</segment>
+<segment>
+<pinref part="IND1" gate="G$1" pin="TESTPOINT"/>
+<pinref part="GND42" gate="1" pin="GND"/>
+<wire x1="160.02" y1="53.34" x2="162.56" y2="53.34" width="0.1524" layer="91"/>
+<wire x1="162.56" y1="53.34" x2="162.56" y2="50.8" width="0.1524" layer="91"/>
 </segment>
 </net>
@@
 <segment>
 <pinref part="JP1" gate="G$1" pin="1"/>
-<pinref part="L6" gate="A" pin="2"/>
 <wire x1="160.02" y1="58.42" x2="172.72" y2="58.42" width="0.1524" layer="91"/>
 <wire x1="172.72" y1="55.88" x2="172.72" y2="58.42" width="0.1524" layer="91"/>
-</segment>
-</net>
+<pinref part="IND" gate="G$1" pin="TESTPOINT"/>
+</segment>
+</net>
