File: powerwatch/electron_rev_4/hardware/plugwatch.brd (EAGLE design)
At the start: 52.8 x 90.9 mm, 143 parts, among them J1 DM3AT-SF-PEJM5, J2 TC2030-JLINK-NL, Q1 SI223DDS, Q2 MOSFET-NCHANNELSMD, U1 BGA725L6-ALT, U10 SIP32510, U11 SIP32510, U12 SIP32510, U14 MPU-9250, U16 MAX6746, U2 SAFFB1G56KB0F0A, U3 IRM-03-5V, U4 MAX-M8, U5 MAX9910, U6 SIP32510, U7 NRF51822QF, U8 MAX9910, U9 SIP32510, X1 32.768k, X2 16MHz

Commit message: add rtc and descriptions, remove BLE
Parts:
- removed A1: ANT3216A063R2400A, chips:ANT3216A063R2400A
- removed B1: BAL-NRF01D3, chips:BAL-NRF01D3
- removed C10: 2.2nF, passives:0402_CAP
- removed C14: 47nF, passives:0402_CAP
- removed C16: 100nF, passives:0402_CAP
- removed C22: 1uF, passives:0402_CAP
- removed C25: 4.7uF, passives:0402_CAP
- removed C4, C5, C6: 12pF, passives:0402_CAP
- removed C8, C9: 1nF, passives:0402_CAP
- removed D2: BLUE, leds:LED-0603
- removed J2: TC2030-JLINK-NL, connector:TC2030-IDC-NL
- removed L2: 15nH, passives:0402_CAP
- removed L3: 10uH, passives:0603_CAP
- removed S1: B3U-1000P, switches:B3U-1000P
- removed TP10, TP11, TP25, TP27, TP7, TP9: TEST_POINT_0.040IN, headers:TESTPOINT_0.040IN
- removed U11: SIP32510, chips:TSOT23-6
- removed U7: NRF51822QF, chips:QFN-48-6MM
- removed X2: 16MHz, crystals:TXC-8Y
- added B2: (no value), batteries:MS518SE-FL35E
- added R32, R33: 1.5k, passives:0402_RES
- added R34: 10k, passives:0402_RES
- added U13: AB1815-T3, chips:QFN-16-3MM
- C1: value 0.8pF -> 1uF; device passives:0402_CAP -> passives:0603_CAP
- C3: value 12pF -> 47pF; device passives:0402_CAP -> passives:0603_CAP
- R15: value 12k -> 100k
- R2: value 150 -> 10k
- R20: value 100k -> 10k
- R5: value 1k -> 100k
- X1: value 32.768k -> ABS07-32.768KHZ-7-T; device crystals:ABS05 -> crystals:2-SMD
- moved R20 347.0 mm to (-96.5, -317.5), flipped to the top, turned to 0 degrees
- moved R5 341.7 mm to (-96.5, -307.3), flipped to the top, turned to 0 degrees
- moved R15 336.6 mm to (-96.5, -312.4), flipped to the top
- moved X1 331.8 mm to (-99.1, -294.6), flipped to the top, turned to 0 degrees
- moved R2 329.1 mm to (-96.5, -302.3), flipped to the top, turned to 0 degrees
- moved C3 327.8 mm to (-88.9, -297.2), flipped to the top, turned to 0 degrees
- moved C1 318.9 mm to (-88.9, -292.1), flipped to the top, turned to 0 degrees
Connections:
- removed net !LIGHT_INT: ASSY1.A1, TP7.TESTPOINT
- removed net AUDIO_OUT: ASSY1.B2, TP11.TESTPOINT
- removed net AUDIO_PWR_EN: ASSY1.B4, TP10.TESTPOINT
- removed net AVDD1: C22.1, C8.1, L2.1, U7.35, U7.36
- removed net A_MIC_OUT: TP27.TESTPOINT
- removed net DCC1: L3.2, U7.2
- removed net N$10: B1.ANT1, U7.31
- removed net N$12: B1.ANT2, U7.32
- removed net N$15: L2.2, L3.1
- removed net N$22: C9.1, U7.39
- removed net N$24: C14.1, U7.29
- removed net N$26: R2.2, S1.2
- removed net NRF_A2: C6.1, U7.46, X1.B
- removed net NRF_A3: C5.1, U7.45, X1.A
- removed net NRF_P29: D2.C, U7.48
- removed net NRF_SWDCLK: J2.4, R15.1, U7.24
- removed net NRF_SWDIO/!RESET: ASSY1.D7, J2.2, R2.1, TP25.TESTPOINT, U7.23
- removed net VCC_BLE: C16.1, C25.1, J2.1, R5.1, U11.1, U11.2, U7.1, U7.12
- removed net VDD_PA1: B1.VCC, C10.1, U7.30
- new net !RTC_CS: U13.12
- new net !RTC_INT1: R34.2, U13.11
- new net !RTC_INT2: R20.2, U13.4
- new net N$4: B2.+, R32.2, R33.1
- new net N$5: R33.2, U13.5
- net 5V: now also R5.1
- net BLE_PWR_EN: no longer R20.2, TP9.TESTPOINT, U11.3
- net BLE_RXD: no longer ASSY1.C3, U7.25
- net BLE_TXD: no longer ASSY1.C2, U7.22
- net GND: now also B2.-, R2.2, U13.3, U13.GND; no longer A1.S2, B1.GND, C10.2, C14.2, C16.2, C22.2, C25.2, C4.2, C5.2, C6.2, C8.2, C9.2, J2.5, R20.1, S1.1, U11.4, U7.13, U7.33, U7.34, U7.GND
- net N$13: now also C3.1, U13.14; no longer A1.S1, B1.SE, C1.1
- net N$20: now also U13.15, X1.2; no longer C3.1, U7.37, X2.1
- net N$21: now also U13.16, X1.1; no longer C4.1, U7.38, X2.3
- net N$25: now also R15.1, U13.10; no longer D2.A
- net SD_MISO: now also U13.6
- net SD_MOSI: now also U13.9
- net SD_SCLK: now also U13.7
- net VCC: now also C1.1, R20.1, R32.1, R34.1, U13.13; no longer U11.5, U11.6
- net WDI: now also R2.1, U13.2
Routing:
- net NRF_SWDIO/!RESET: track 74.0 -> 0.00 mm, vias 1 -> 0
- net AUDIO_OUT: track 61.3 -> 0.00 mm, vias 1 -> 0
- net AUDIO_PWR_EN: track 59.0 -> 0.00 mm
- net !LIGHT_INT: track 46.6 -> 0.00 mm, vias 1 -> 0
- net VCC_BLE: track 27.8 -> 0.00 mm, vias 2 -> 0
- net BLE_TXD: track 93.5 -> 67.9 mm
- net BLE_RXD: track 85.7 -> 60.4 mm
- net AVDD1: track 17.1 -> 0.00 mm, vias 2 -> 0
- net A_MIC_OUT: track 15.3 -> 0.00 mm
- net GND: track 53.1 -> 43.5 mm, vias 208 -> 205
- net NRF_SWDCLK: track 7.63 -> 0.00 mm, vias 1 -> 0
- net N$13: track 6.63 -> 0.00 mm
- net NRF_P29: track 5.40 -> 0.00 mm
- net NRF_A3: track 5.15 -> 0.00 mm
- net NRF_A2: track 4.97 -> 0.00 mm
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
Commit message: add mic, remove many old things, connect RTC, new Accel
Parts:
- removed C18: 100nF, passives:0402_CAP
- removed D3: BLUE, leds:LED-0603
- removed S2: PTS645SM43SMTR92, switches:PTS645
- removed U14: MPU-9250, chips:QFN-24/3MM
- added R35: 66.5, passives:0402_RES
- added R36: 34k, passives:0402_RES
- added TP10, TP11, TP7, TP9: TEST_POINT_0.040IN, headers:TESTPOINT_0.040IN
- added U7: (no value), microphones:SPH0465
- C13: value 10nF -> 10uF
- C19: value 100nF -> 0.1uF
- R11: value 10k -> 68
- R26: value 100k -> 68
- R3: value 150 -> 68
- R6: value 1k -> 10k
- U6: value SIP32510 -> LIS2DW12; device chips:TSOT23-6 -> chips:LGA-12
- moved C1 342.9 mm to (-83.8, 50.8)
- moved R15 342.9 mm to (-91.4, 30.5)
- moved C3 342.9 mm to (-83.8, 45.7)
- moved R2 342.9 mm to (-91.4, 40.6)
- moved R20 342.9 mm to (-91.4, 25.4)
- moved R34 342.9 mm to (-91.4, 20.3)
- moved R5 342.9 mm to (-91.4, 35.6)
- moved X1 342.9 mm to (-94.0, 48.3)
- moved B2 283.0 mm to (10.2, -12.7)
- moved R32 275.7 mm to (-61.0, -7.62)
- moved R33 275.7 mm to (-61.0, -12.7)
- moved D11 226.4 mm to (-68.6, -30.5)
- moved C100 226.4 mm to (-71.1, 40.6)
- moved C101 226.4 mm to (-68.6, 15.2)
- moved D10 226.4 mm to (-68.6, -25.4)
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Connections:
- removed net !IMU_INT: ASSY1.D2, R11.1, TP21.TESTPOINT, U14.12
- removed net !SAFEMODE: TP8.TESTPOINT
- removed net !SOFT_RST: ASSY1.A0, R3.2, S2.3, S2.4
- removed net !WIFI_RESET: ASSY1.C4, ASSY2.6, TP17.TESTPOINT
- removed net BLE_PWR_EN: ASSY1.B5
- removed net BLE_RXD: TP16.TESTPOINT
- removed net BLE_TXD: TP15.TESTPOINT
- removed net LED: ASSY1.C5, D3.C
- removed net N$19: C18.1, U14.10
- removed net N$30: R26.1, U6.4
- removed net SENSORS_PWR_EN: ASSY1.B3, R26.2, U6.3
- removed net VCC_SENSORS: C13.1, C19.1, R10.2, R11.2, R9.2, U14.1, U14.13, U14.22, U14.8, U6.1, U6.2
- new net ACCEL_INT: ASSY1.C4, TP21.TESTPOINT, U6.12
- new net MIC_BCLK: ASSY1.D4, R11.2, TP10.TESTPOINT
- new net MIC_DATA: ASSY1.D2, R26.1, TP9.TESTPOINT
- new net MIC_WS: ASSY1.D5, R3.2, TP8.TESTPOINT
- new net N$10: ASSY1.WKP, R35.1, R36.2
- new net N$12: R11.1, U7.4
- new net N$15: R26.2, U7.6
- net !EXTERNAL_RST: now also TP17.TESTPOINT
- net !GPS_RESET: now also ASSY1.C3; no longer ASSY1.D4
- net !RTC_CS: now also ASSY1.C5, R6.2, TP11.TESTPOINT
- net !RTC_INT1: now also ASSY1.D7, TP15.TESTPOINT
- net 5V: now also R36.1
- net AC/L-MEASURE: now also ASSY1.B5
- net AC/L-PERTURB: now also ASSY1.A0
- net AC/L-SENSE: now also ASSY1.B4
- net AC/N-MEASURE: now also ASSY1.B3
- net AC/N-PERTURB: now also ASSY1.A1
- net AC/N-SENSE: now also ASSY1.B2
- net GND: now also R35.2, U6.3, U6.5, U6.6, U6.7, U6.8, U7.3; no longer C18.2, S2.1, S2.2, U14.11, U14.18, U14.20, U14.9
- net N$14: now also ASSY2.6
- net N$3: now also R3.1, U7.1; no longer D3.A, R6.2
- net SD_ENABLE: now also ASSY1.C2, TP7.TESTPOINT; no longer ASSY1.D5
- net SENSORS_SCL: now also R9.1, U6.1; no longer R10.1, U14.23
- net SENSORS_SDA: now also R10.1, U6.4; no longer R9.1, U14.24
- net VCC: now also C13.1, C19.1, R10.2, R9.2, U6.10, U6.2, U6.9, U7.2, U7.5; no longer R3.1, U6.5, U6.6
- net WDI: now also TP16.TESTPOINT
Routing:
- net VCC_SENSORS: track 109.6 -> 0.00 mm, vias 8 -> 0
- net BLE_PWR_EN: track 86.6 -> 0.00 mm, vias 1 -> 0
- net BLE_TXD: track 67.9 -> 0.00 mm, vias 1 -> 0
- net BLE_RXD: track 60.4 -> 0.00 mm, vias 1 -> 0
- net !SAFEMODE: track 59.8 -> 0.00 mm
- net !IMU_INT: track 36.5 -> 0.00 mm
- net !WIFI_RESET: track 30.7 -> 0.00 mm
- net LED: track 27.0 -> 0.00 mm
- net ACCEL_INT: track 0.00 -> 21.7 mm
- net !GPS_RESET: track 47.5 -> 33.8 mm
- net !SOFT_RST: track 9.84 -> 0.00 mm
- net VCC: track 55.2 -> 46.7 mm, vias 6 -> 3
- net SD_ENABLE: track 34.0 -> 25.9 mm
- net SENSORS_SCL: track 76.0 -> 69.5 mm
- net SENSORS_SDA: track 90.5 -> 84.7 mm
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- removed copper zone on layer 15, net N$33
- removed copper zone on layer 16, net N$34
- removed copper zone on layer 1, net N$37
Other:
- board text removed: "!IMU_INT"
- board text removed: "!LIGHT_INT"
- board text removed: "!WIFI_RESET"
- board text removed: "(ON, ON)"
- board text removed: "APN"
- board text removed: "AUDIO"
- board text removed: "AUDIO_OUT"
- board text removed: "AUDIO_PWR_EN"
- board text removed: "BLE PROG"
- board text removed: "BLE_PWR_EN"
- board text removed: "BRD_ANT"
- board text removed: "IND_ANT"
- board text removed: "MIC PRE-FILT"
- board text removed: "NRF_SWDIO/ !RESET"
- board text removed: "RESET"

Commit message: started rough section layout
Parts:
- moved U13 163.5 mm to (35.6, 73.7)
- moved R11 160.0 mm to (38.1, 66.0)
- moved R3 157.8 mm to (40.6, 63.5)
- moved R26 152.4 mm to (38.1, 68.6)
- moved U7 150.3 mm to (43.2, 66.0)
- moved R6 148.8 mm to (43.2, 63.5)
- moved U6 139.8 mm to (35.6, 63.5)
- moved R36 139.1 mm to (38.1, 61.0)
- moved R15 138.6 mm to (43.2, 63.5)
- moved R20 137.5 mm to (40.6, 63.5)
- moved X1 137.0 mm to (40.6, 73.7)
- moved R35 135.9 mm to (35.6, 63.5)
- moved R34 133.3 mm to (35.6, 61.0)
- moved R2 131.5 mm to (38.1, 63.5)
- moved R5 129.5 mm to (35.6, 61.0)
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Routing:
- net SENSORS_SCL: track 69.5 -> 1.94 mm
- net SENSORS_SDA: track 84.7 -> 22.7 mm
- net !SD_CS: track 62.5 -> 2.76 mm
- net SD_MISO: track 65.9 -> 6.63 mm
- net SD_SCLK: track 55.8 -> 0.69 mm, vias 1 -> 2
- net WIFI_PWR_EN: track 59.5 -> 12.9 mm
- net SD_MOSI: track 51.7 -> 5.78 mm, vias 1 -> 2
- net !SD_DETECT: track 60.0 -> 16.9 mm
- net GND: track 42.5 -> 5.05 mm, vias 106 -> 22
- net VCC: track 46.7 -> 10.8 mm, vias 3 -> 2
- net GPS_PWR_EN: track 36.1 -> 6.30 mm, vias 1 -> 0
- net GPS_TXD: track 30.6 -> 1.60 mm
- net GPS_RXD: track 28.8 -> 0.00 mm
- net SERIAL_NUM: track 27.4 -> 0.00 mm
- net !GPS_RESET: track 33.8 -> 7.07 mm
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Other:
- board text removed: "!GPS_RESET"
- board text removed: "!SAFEMODE"
- board text removed: "!SD_CS"
- board text removed: "BLE_RXD"
- board text removed: "BLE_TXD"
- board text removed: "GND"
- board text removed: "GPS_PWR_EN"
- board text removed: "GPS_RXD"
- board text removed: "GPS_TXD"
- board text removed: "SD CARD"
- board text removed: "SD_DETECT"
- board text removed: "SD_MISO"
- board text removed: "SD_MOSI"
- board text removed: "SD_SCLK"
- board text removed: "SENSE_SDA"
- board text removed: "SENSORS_SCL"
- board text removed: "S_NUM"
- board text removed: "USB"
- board text removed: "VCC"
- board text removed: "WIFI_PWR_EN"
- board text removed: "WIFI_RXD"

Commit message: switch the gnd float mosfet?
Connections:
- removed net N$9: C17.2, C2.-, C7.2, Q2.3, U3.V-
- new net N$8: Q2.2, U3.V-
- net GND: now also C17.2, C2.-, C7.2, Q2.3; no longer Q2.2
Changed lines of the file:
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@@
 <contactref element="C29" pad="2"/>
 <contactref element="R27" pad="2"/>
-<contactref element="Q2" pad="2"/>
 <contactref element="R23" pad="1"/>
 <contactref element="C100" pad="2"/>
@@
 <contactref element="U7" pad="3"/>
 <via x="42.113" y="50.851" extent="1-16" drill="0.4064"/>
+<contactref element="C2" pad="-"/>
+<contactref element="C7" pad="2"/>
+<contactref element="C17" pad="2"/>
+<contactref element="Q2" pad="3"/>
 <wire x1="35.56" y1="73.66" x2="37.084" y2="83.567" width="0" layer="19" extent="1-1"/>
 <wire x1="34.16" y1="73.41" x2="35.56" y2="73.66" width="0" layer="19" extent="1-1"/>
@@
 <wire x1="40.09" y1="60.96" x2="38.75" y2="60.96" width="0" layer="19" extent="1-1"/>
 <wire x1="36.21" y1="58.42" x2="38.75" y2="60.96" width="0" layer="19" extent="1-1"/>
+<wire x1="35.89" y1="55.78" x2="36.21" y2="58.42" width="0" layer="19" extent="1-16"/>
 <wire x1="43.61306875" y1="63.5" x2="40.09" y2="60.96" width="0" layer="19" extent="1-1"/>
 <wire x1="43.18" y1="65.33" x2="43.61306875" y2="63.5" width="0" layer="19" extent="1-1"/>
+<wire x1="38.862" y1="52.07" x2="35.89" y2="55.78" width="0" layer="19" extent="1-16"/>
+<wire x1="39.5732" y1="52.75453125" x2="38.862" y2="52.07" width="0" layer="19" extent="1-1"/>
+<wire x1="42.94" y1="55.78" x2="40.894" y2="52.07" width="0" layer="19" extent="16-16"/>
+<wire x1="46.09" y1="55.78" x2="42.94" y2="55.78" width="0" layer="19" extent="16-16"/>
+<wire x1="47.04" y1="51.48" x2="46.09" y2="55.78" width="0" layer="19" extent="16-16"/>
 <wire x1="44.44" y1="70.37" x2="43.18" y2="65.33" width="0" layer="19" extent="1-1"/>
+<wire x1="42.164" y1="43.688" x2="42.113" y2="50.851" width="0" layer="19" extent="1-1"/>
+<wire x1="41.148" y1="43.50893125" x2="42.164" y2="43.688" width="0" layer="19" extent="1-1"/>
+<wire x1="47.04" y1="41.13" x2="42.164" y2="43.688" width="0" layer="19" extent="16-16"/>
+<wire x1="48.6918" y1="40.5892" x2="47.04" y2="41.13" width="0" layer="19" extent="16-16"/>
+<wire x1="48.514" y1="34.29" x2="48.6918" y2="40.5892" width="0" layer="19" extent="1-1"/>
+<wire x1="44.77" y1="34.65425" x2="48.514" y2="34.29" width="0" layer="19" extent="16-16"/>
+<wire x1="49.53" y1="27.432" x2="48.514" y2="34.29" width="0" layer="19" extent="1-1"/>
+<wire x1="52.07" y1="23.44293125" x2="49.53" y2="27.432" width="0" layer="19" extent="16-16"/>
+<wire x1="53.594" y1="23.622" x2="52.07" y2="23.44293125" width="0" layer="19" extent="16-16"/>
+<wire x1="53.594" y1="22.606" x2="53.594" y2="23.622" width="0" layer="19" extent="1-1"/>
+<wire x1="33.54" y1="40.68" x2="41.148" y2="43.50893125" width="0" layer="19" extent="1-16"/>
+<wire x1="30.9118" y1="45.6692" x2="33.54" y2="40.68" width="0" layer="19" extent="16-16"/>
+<wire x1="46.66106875" y1="16.256" x2="52.07" y2="23.44293125" width="0" layer="19" extent="16-16"/>
+<wire x1="46.66106875" y1="15.24" x2="46.66106875" y2="16.256" width="0" layer="19" extent="16-16"/>
+<wire x1="40.894" y1="14.224" x2="46.66106875" y2="15.24" width="0" layer="19" extent="16-16"/>
+<wire x1="26.56" y1="80.28" x2="26.162" y2="70.104" width="0" layer="19" extent="1-1"/>
+<wire x1="26.05" y1="88.9" x2="26.56" y2="80.28" width="0" layer="19" extent="1-1"/>
+<wire x1="25.83306875" y1="88.9" x2="26.05" y2="88.9" width="0" layer="19" extent="1-1"/>
+<wire x1="27.94" y1="90" x2="26.05" y2="88.9" width="0" layer="19" extent="1-1"/>
+<wire x1="23.51" y1="88.9" x2="25.83306875" y2="88.9" width="0" layer="19" extent="1-1"/>
+<wire x1="18.755" y1="87.73" x2="23.51" y2="88.9" width="0" layer="19" extent="1-1"/>
+<wire x1="11.54" y1="82.28" x2="18.755" y2="87.73" width="0" layer="19" extent="1-1"/>
 <wire x1="12.268" y1="61.386" x2="22.298" y2="59.274" width="0" layer="19" extent="1-16"/>
 <wire x1="9.198" y1="59.274" x2="12.268" y2="61.386" width="0" layer="19" extent="1-16"/>
@@
 <wire x1="1.92175" y1="66.614" x2="6.096" y2="67.63893125" width="0" layer="19" extent="16-16"/>
 <wire x1="0.508" y1="68.50506875" x2="1.92175" y2="66.614" width="0" layer="19" extent="16-16"/>
-<wire x1="26.56" y1="80.28" x2="9.198" y2="70.774" width="0" layer="19" extent="1-1"/>
-<wire x1="11.54" y1="82.28" x2="26.56" y2="80.28" width="0" layer="19" extent="1-1"/>
-<wire x1="18.755" y1="87.73" x2="26.56" y2="80.28" width="0" layer="19" extent="1-1"/>
-<wire x1="23.51" y1="88.9" x2="18.755" y2="87.73" width="0" layer="19" extent="1-1"/>
-<wire x1="25.83306875" y1="88.9" x2="23.51" y2="88.9" width="0" layer="19" extent="1-1"/>
-<wire x1="28.89" y1="87.9" x2="25.83306875" y2="88.9" width="0" layer="19" extent="1-1"/>
-<wire x1="26.05" y1="88.9" x2="28.89" y2="87.9" width="0" layer="19" extent="1-1"/>
-<wire x1="30.9118" y1="45.6692" x2="19.37" y2="40.64" width="0" layer="19" extent="1-1"/>
-<wire x1="47.04" y1="41.13" x2="0.508" y2="68.50506875" width="0" layer="19" extent="16-16"/>
-<wire x1="47.04" y1="51.48" x2="47.04" y2="41.13" width="0" layer="19" extent="16-16"/>
-<wire x1="46.09" y1="55.78" x2="47.04" y2="51.48" width="0" layer="19" extent="16-16"/>
-<wire x1="42.113" y1="50.851" x2="46.09" y2="55.78" width="0" layer="19" extent="1-16"/>
-<wire x1="39.5732" y1="52.75453125" x2="38.862" y2="52.07" width="0" layer="19" extent="1-1"/>
-<wire x1="42.94" y1="55.78" x2="42.113" y2="50.851" width="0" layer="19" extent="1-16"/>
-<wire x1="42.164" y1="43.688" x2="42.94" y2="55.78" width="0" layer="19" extent="16-16"/>
-<wire x1="41.148" y1="43.50893125" x2="42.164" y2="43.688" width="0" layer="19" extent="1-1"/>
-<wire x1="35.89" y1="55.78" x2="42.164" y2="43.688" width="0" layer="19" extent="16-16"/>
-<wire x1="33.54" y1="40.68" x2="47.04" y2="41.13" width="0" layer="19" extent="16-16"/>
-<wire x1="44.77" y1="34.65425" x2="30.9118" y2="45.6692" width="0" layer="19" extent="16-16"/>
-<wire x1="48.514" y1="34.29" x2="44.77" y2="34.65425" width="0" layer="19" extent="16-16"/>
-<wire x1="48.6918" y1="40.5892" x2="48.514" y2="34.29" width="0" layer="19" extent="1-1"/>
-<wire x1="49.53" y1="27.432" x2="48.514" y2="34.29" width="0" layer="19" extent="1-1"/>
-<wire x1="52.07" y1="23.44293125" x2="49.53" y2="27.432" width="0" layer="19" extent="16-16"/>
-<wire x1="53.594" y1="23.622" x2="52.07" y2="23.44293125" width="0" layer="19" extent="16-16"/>
-<wire x1="53.594" y1="22.606" x2="53.594" y2="23.622" width="0" layer="19" extent="1-1"/>
-<wire x1="46.66106875" y1="16.256" x2="52.07" y2="23.44293125" width="0" layer="19" extent="16-16"/>
-<wire x1="46.66106875" y1="15.24" x2="46.66106875" y2="16.256" width="0" layer="19" extent="16-16"/>
-<wire x1="40.894" y1="14.224" x2="46.66106875" y2="15.24" width="0" layer="19" extent="16-16"/>
+<wire x1="25.4" y1="10.16" x2="23.96" y2="22.86" width="0" layer="19" extent="1-1"/>
+<wire x1="16.79" y1="10.16" x2="25.4" y2="10.16" width="0" layer="19" extent="1-1"/>
+<wire x1="14.25" y1="7.62" x2="16.79" y2="10.16" width="0" layer="19" extent="1-1"/>
 <wire x1="-12.7" y1="28.194" x2="11.26" y2="27.94" width="0" layer="19" extent="1-1"/>
 </signal>
@@
 <wire x1="37.66693125" y1="60.96" x2="35.12693125" y2="60.96" width="0" layer="19" extent="1-1"/>
 </signal>
-<signal name="N$9">
-<contactref element="U3" pad="V-"/>
-<contactref element="C2" pad="-"/>
-<contactref element="C7" pad="2"/>
-<contactref element="C17" pad="2"/>
-<contactref element="Q2" pad="3"/>
-<wire x1="14.25" y1="7.62" x2="16.79" y2="10.16" width="0" layer="19" extent="1-1"/>
-<wire x1="25.4" y1="10.16" x2="14.25" y2="7.62" width="0" layer="19" extent="1-1"/>
-<wire x1="22.352" y1="52.324" x2="25.4" y2="10.16" width="0" layer="19" extent="1-1"/>
-<wire x1="27.94" y1="90" x2="16.79" y2="10.16" width="0" layer="19" extent="1-1"/>
-</signal>
 <signal name="N$32">
+<contactref element="R1" pad="2"/>
 <contactref element="Q2" pad="1"/>
-<contactref element="R1" pad="2"/>
 <wire x1="26.99" y1="87.9" x2="23.29306875" y2="88.9" width="0" layer="19" extent="1-1"/>
 </signal>
@@
 <wire x1="30.9118" y1="53.2892" x2="41.07306875" y2="63.5" width="0" layer="19" extent="1-1"/>
 </signal>
+<signal name="N$8">
+<contactref element="U3" pad="V-"/>
+<contactref element="Q2" pad="2"/>
+<wire x1="22.352" y1="52.324" x2="28.89" y2="87.9" width="0" layer="19" extent="1-1"/>
+</signal>
 </signals>
